File: Power.sch (KiCad schematic (older format))
At the start: 0 parts

Commit message: added LiPo charging circuit
Parts:
- added C10, C11: 4.7uF, symbol Device:C
- added D10: LED, symbol Device:LED
- added J10: Conn_01x02_Female, symbol Connector:Conn_01x02_Female
- added R10: 2kR, Resistor_SMD:R_0402_1005Metric_Pad0.72x0.64mm_HandSolder, symbol Device:R
- added R11: 470R, Resistor_SMD:R_1206_3216Metric_Pad1.30x1.75mm_HandSolder, symbol Device:R
- added U3: MCP73831T-2ACI_OT, digikey-footprints:SOT-753, symbol dk_PMIC-Battery-Chargers:MCP73831T-2ACI_OT
Connections:
- new net: R10.1, U3.5 (PROG)
- new net: D10.1 (K), R11.1
- new net: R11.2, U3.1 (STAT)
- new net 5V: C11.1, D10.2 (A), U3.4 (VDD)
- new net GND: C10.2, C11.2, J10.2 (Pin_2), R10.2, U3.2 (VSS)
- new net VBatt: C10.1, J10.1 (Pin_1), U3.3 (VBAT)
Changed lines of the file:
@@
 $Descr A4 11693 8268
 encoding utf-8
-Sheet 1 3
+Sheet 1 1
 Title ""
 Date ""
@@
 Comment4 ""
 $EndDescr
+$Comp
+L dk_PMIC-Battery-Chargers:MCP73831T-2ACI_OT U3
+U 1 1 5FBBC2AA
+P 3400 2850
+F 0 "U3" H 3150 3000 60  0000 C CNN
+F 1 "MCP73831T-2ACI_OT" H 3500 2450 60  0000 C CNN
+F 2 "digikey-footprints:SOT-753" H 3600 3050 60  0001 L CNN
+F 3 "http://ww1.microchip.com/downloads/en/DeviceDoc/20001984g.pdf" H 3600 3150 60  0001 L CNN
+F 4 "MCP73831T-2ACI/OTCT-ND" H 3600 3250 60  0001 L CNN "Digi-Key_PN"
+F 5 "MCP73831T-2ACI/OT" H 3600 3350 60  0001 L CNN "MPN"
+F 6 "Integrated Circuits (ICs)" H 3600 3450 60  0001 L CNN "Category"
+F 7 "PMIC - Battery Chargers" H 3600 3550 60  0001 L CNN "Family"
+F 8 "http://ww1.microchip.com/downloads/en/DeviceDoc/20001984g.pdf" H 3600 3650 60  0001 L CNN "DK_Datasheet_Link"
+F 9 "/product-detail/en/microchip-technology/MCP73831T-2ACI-OT/MCP73831T-2ACI-OTCT-ND/1979802" H 3600 3750 60  0001 L CNN "DK_Detail_Page"
+F 10 "IC CONTROLLR LI-ION 4.2V SOT23-5" H 3600 3850 60  0001 L CNN "Description"
+F 11 "Microchip Technology" H 3600 3950 60  0001 L CNN "Manufacturer"
+F 12 "Active" H 3600 4050 60  0001 L CNN "Status"
+	1    3400 2850
+	1    0    0    -1
+$EndComp
+Text HLabel 4200 2850 2    50   Input ~ 0
+VBatt
+Text HLabel 4100 1900 2    50   Input ~ 0
+5V
+Wire Wire Line
+	3400 3250 3400 3400
+$Comp
+L power:GND #PWR?
+U 1 1 5FB4B96A
+P 3400 3400
+F 0 "#PWR?" H 3400 3150 50  0001 C CNN
+F 1 "GND" H 3405 3227 50  0000 C CNN
+F 2 "" H 3400 3400 50  0001 C CNN
+F 3 "" H 3400 3400 50  0001 C CNN
+	1    3400 3400
+	1    0    0    -1
+$EndComp
+Wire Wire Line
+	3800 2850 4100 2850
+Wire Wire Line
+	4100 2850 4100 3000
+Connection ~ 4100 2850
+Wire Wire Line
+	4100 2850 4200 2850
+$Comp
+L Device:C C10
+U 1 1 5FB4BFE1
+P 4100 3150
+F 0 "C10" H 4215 3196 50  0000 L CNN
+F 1 "4.7uF" H 4215 3105 50  0000 L CNN
+F 2 "" H 4138 3000 50  0001 C CNN
+F 3 "~" H 4100 3150 50  0001 C CNN
+	1    4100 3150
+	1    0    0    -1
+$EndComp
+$Comp
+L power:GND #PWR?
+U 1 1 5FB4C6F8
+P 4100 3400
+F 0 "#PWR?" H 4100 3150 50  0001 C CNN
+F 1 "GND" H 4105 3227 50  0000 C CNN
+F 2 "" H 4100 3400 50  0001 C CNN
+F 3 "" H 4100 3400 50  0001 C CNN
+	1    4100 3400
+	1    0    0    -1
+$EndComp
+Wire Wire Line
+	4100 3300 4100 3400
+Wire Wire Line
+	3000 2950 2850 2950
+Wire Wire Line
+	2850 2950 2850 3050
+$Comp
+L Device:R R10
+U 1 1 5FB4CE98
+P 2850 3200
+F 0 "R10" H 2700 3350 50  0000 L CNN
+F 1 "2kR" V 2850 3150 50  0000 L CNN
+F 2 "Resistor_SMD:R_0402_1005Metric_Pad0.72x0.64mm_HandSolder" V 2780 3200 50  0001 C CNN
+F 3 "https://www.digikey.com/en/products/detail/bourns-inc/CR0402AFX-2001GLF/12091352" H 2850 3200 50  0001 C CNN
+	1    2850 3200
+	1    0    0    -1
+$EndComp
+Wire Wire Line
+	2850 3350 2850 3400
+$Comp
+L power:GND #PWR?
+U 1 1 5FB4D469
+P 2850 3400
+F 0 "#PWR?" H 2850 3150 50  0001 C CNN
+F 1 "GND" H 2855 3227 50  0000 C CNN
+F 2 "" H 2850 3400 50  0001 C CNN
+F 3 "" H 2850 3400 50  0001 C CNN
+	1    2850 3400
+	1    0    0    -1
+$EndComp
+Wire Wire Line
+	4100 1900 4100 2050
+$Comp
+L Device:C C11
+U 1 1 5FB4F413
+P 4100 2200
+F 0 "C11" H 4215 2246 50  0000 L CNN
+F 1 "4.7uF" H 4215 2155 50  0000 L CNN
+F 2 "" H 4138 2050 50  0001 C CNN
+F 3 "~" H 4100 2200 50  0001 C CNN
+	1    4100 2200
+	1    0    0    -1
+$EndComp
+$Comp
+L power:GND #PWR?
+U 1 1 5FB4F419
+P 4100 2450
+F 0 "#PWR?" H 4100 2200 50  0001 C CNN
+F 1 "GND" H 4105 2277 50  0000 C CNN
+F 2 "" H 4100 2450 50  0001 C CNN
+F 3 "" H 4100 2450 50  0001 C CNN
+	1    4100 2450
+	1    0    0    -1
+$EndComp
+Wire Wire Line
+	4100 2350 4100 2450
+Wire Wire Line
+	3400 1900 3400 2650
+Wire Wire Line
+	4100 1900 3850 1900
+Wire Wire Line
+	3850 2300 3850 2450
+Wire Wire Line
+	3850 2000 3850 1900
+$Comp
+L Device:LED D10
+U 1 1 5FB5074E
+P 3850 2150
+F 0 "D10" V 3950 2300 50  0000 R CNN
+F 1 "LED" V 3750 2350 50  0000 R CNN
+F 2 "" H 3850 2150 50  0001 C CNN
+F 3 "~" H 3850 2150 50  0001 C CNN
+	1    3850 2150
+	0    -1   -1   0
+$EndComp
+$Comp
+L Device:R R11
+U 1 1 5FB5016C
+P 3850 2600
+F 0 "R11" H 3650 2550 50  0000 L CNN
+F 1 "470R" H 3600 2650 50  0000 L CNN
+F 2 "Resistor_SMD:R_1206_3216Metric_Pad1.30x1.75mm_HandSolder" V 3780 2600 50  0001 C CNN
+F 3 "https://www.digikey.com/en/products/detail/vishay-dale/CRCW1206470RFKEAC/7920591" H 3850 2600 50  0001 C CNN
+	1    3850 2600
+	1    0    0    -1
+$EndComp
+Connection ~ 3850 1900
+Wire Wire Line
+	3400 1900 3850 1900
+Wire Wire Line
+	3800 2950 3850 2950
+Wire Wire Line
+	3850 2950 3850 2750
+Wire Wire Line
+	4100 2850 4100 2750
+Wire Wire Line
+	4100 2750 4650 2750
+$Comp
+L Connector:Conn_01x02_Female J10
+U 1 1 5FB56977
+P 4850 2750
+F 0 "J10" H 4878 2726 50  0000 L CNN
+F 1 "Conn_01x02_Female" H 4878 2635 50  0000 L CNN
+F 2 "" H 4850 2750 50  0001 C CNN
+F 3 "~" H 4850 2750 50  0001 C CNN
+	1    4850 2750
+	1    0    0    -1
+$EndComp
+Wire Wire Line
+	4650 2850 4600 2850
+Wire Wire Line
+	4600 2850 4600 2950
+$Comp
+L power:GND #PWR?
+U 1 1 5FB57A73
+P 4600 2950
+F 0 "#PWR?" H 4600 2700 50  0001 C CNN
+F 1 "GND" H 4605 2777 50  0000 C CNN
+F 2 "" H 4600 2950 50  0001 C CNN
+F 3 "" H 4600 2950 50  0001 C CNN
+	1    4600 2950
+	1    0    0    -1
+$EndComp
+Text HLabel 4600 2950 2    50   Input ~ 0
+GND
 $EndSCHEMATC
