File: Sensors.sch (KiCad schematic (older format))
At the start: 0 parts

Commit message: REAL COMMIT: Completed initial schematic. Added ADCs, Haptic FB circuits, test points, USB/Battery selection circuits.
Parts:
- added C10, C7, C8: 0.1u, Capacitors_SMD:C_0603_HandSoldering, symbol Device:C
- added C11, C9: 10u, Capacitors_SMD:C_0603_HandSoldering, symbol Device:C
- added D8, D9: SS54, Diode_SMD:D_SMA_Handsoldering, symbol Device:D_Schottky
- added IC2, IC3: MAX11128ATI+, SamacSys_Parts:QFN50P500X500X80-29N, symbol SamacSys_Parts:MAX11128ATI+
- added J5, J6: Conn_01x02_Female, Connector_JST:JST_PH_B2B-PH-SM4-TB_1x02_P2.00mm_Vertical, symbol Connector:Conn_01x02_Female
- added JP1, JP10, JP11, JP12, JP13, JP14, JP15, JP16, JP17, JP18, JP19, JP2, JP20, JP21, JP22, JP23, JP24, JP25, JP26, JP27, JP28, JP29, JP3, JP30, JP31, JP32, JP4, JP5, JP6, JP7, JP8, JP9: SolderJumper_2_Open, Jumper:SolderJumper-2_P1.3mm_Open_RoundedPad1.0x1.5mm, symbol Jumper:SolderJumper_2_Open
- added Q2, Q3: BSS138, Package_TO_SOT_SMD:SOT-23, symbol Transistor_FET:BSS138
- added U2: REF3030, Package_TO_SOT_SMD:SOT-23, symbol Reference_Voltage:REF3030
Connections:
- new net: D8.2 (A), J5.2 (Pin_2), Q2.3 (D)
- new net: D9.2 (A), J6.2 (Pin_2), Q3.3 (D)
- new net +3V3: C10.1, C11.1, C8.1, C9.1, D8.1 (K), D9.1 (K), IC2.17 (VDD_1), IC2.18 (VDD_2), IC2.23 (OVDD), IC3.17 (VDD_1), IC3.18 (VDD_2), IC3.23 (OVDD), J5.1 (Pin_1), J6.1 (Pin_1), U2.1 (IN)
- new net A0: IC2.26 (AIN0), IC3.26 (AIN0)
- new net A1: IC2.27 (AIN1), IC3.27 (AIN1)
- new net A10: JP19.1 (A), JP4.1 (A)
- new net A11: JP20.1 (A), JP5.1 (A)
- new net A12: JP21.1 (A), JP6.1 (A)
- new net A13: JP22.1 (A), JP7.1 (A)
- new net A14: JP23.1 (A), JP8.1 (A)
- new net A15: JP24.1 (A), JP9.1 (A)
- new net A2: IC2.28 (AIN2), IC3.28 (AIN2)
- new net A3: IC2.1 (AIN3), IC3.1 (AIN3)
- new net A4: IC2.2 (AIN4), IC3.2 (AIN4)
- new net A5: IC2.3 (AIN5), IC3.3 (AIN5)
- new net A6: IC2.4 (AIN6), IC3.4 (AIN6)
- new net A7: IC2.5 (AIN7), IC3.5 (AIN7)
- new net A8: JP17.1 (A), JP2.1 (A)
- new net A9: JP18.1 (A), JP3.1 (A)
- new net AIN10_0: IC2.8 (AIN10), JP11.1 (A), JP4.2 (B)
- new net AIN10_1: IC3.8 (AIN10), JP19.2 (B), JP27.1 (A)
- new net AIN11_0: IC2.9 (AIN11), JP12.1 (A), JP5.2 (B)
- new net AIN11_1: IC3.9 (AIN11), JP20.2 (B), JP28.1 (A)
- new net AIN12_0: IC2.10 (AIN12), JP13.1 (A), JP6.2 (B)
- new net AIN12_1: IC3.10 (AIN12), JP21.2 (B), JP29.1 (A)
- new net AIN13_0: IC2.11 (AIN13), JP14.1 (A), JP7.2 (B)
- new net AIN13_1: IC3.11 (AIN13), JP22.2 (B), JP30.1 (A)
- new net AIN14_0: IC2.12 (~CNVST~/AIN14), JP15.1 (A), JP8.2 (B)
- new net AIN14_1: IC3.12 (~CNVST~/AIN14), JP23.2 (B), JP31.1 (A)
- new net AIN15_0: IC2.13 (REF-/AIN15), JP16.1 (A), JP9.2 (B)
- new net AIN15_1: IC3.13 (REF-/AIN15), JP24.2 (B), JP32.1 (A)
- new net AIN8_0: IC2.6 (AIN8), JP1.1 (A), JP2.2 (B)
- new net AIN8_1: IC3.6 (AIN8), JP17.2 (B), JP25.1 (A)
- new net AIN9_0: IC2.7 (AIN9), JP10.1 (A), JP3.2 (B)
- new net AIN9_1: IC3.7 (AIN9), JP18.2 (B), JP26.1 (A)
- new net AREF_3V0: C7.1, IC2.15 (REF+), IC3.15 (REF+), U2.2 (OUT)
- new net GND: C10.2, C11.2, C7.2, C8.2, C9.2, IC2.14 (GND_1), IC2.16 (GND_2), IC2.22 (DGND), IC2.29 (EP), IC3.14 (GND_1), IC3.16 (GND_2), IC3.22 (DGND), IC3.29 (EP), JP1.2 (B), JP10.2 (B), JP11.2 (B), JP12.2 (B), JP13.2 (B), JP14.2 (B), JP15.2 (B), JP16.2 (B), JP25.2 (B), JP26.2 (B), JP27.2 (B), JP28.2 (B), JP29.2 (B), JP30.2 (B), JP31.2 (B), JP32.2 (B), Q2.2 (S), Q3.2 (S), U2.3 (GND)
- new net Haptic_On_0: Q2.1 (G)
- new net Haptic_On_1: Q3.1 (G)
- new net MISO: IC2.24 (DOUT), IC3.24 (DOUT)
- new net MOSI: IC2.21 (DIN), IC3.21 (DIN)
- new net SCK: IC2.19 (SCLK), IC3.19 (SCLK)
- new net ~CS0: IC2.20 (~CS)
- new net ~CS1: IC3.20 (~CS)
- new net ~EOC0: IC2.25 (~EOC)
- new net ~EOC1: IC3.25 (~EOC)
