File: Glove PCB.sch (KiCad schematic (older format))
At the start: 13 parts, among them J1 USB_B_Micro, U1 MDBT50Q-1M

Commit message: REAL COMMIT: Completed initial schematic. Added ADCs, Haptic FB circuits, test points, USB/Battery selection circuits.
Parts:
- removed C3: 10uF, Capacitor_SMD:C_0603_1608Metric_Pad1.08x0.95mm_HandSolder, symbol Device:C
- removed U1: MDBT50Q-1M, symbol Glove_PCB:MDBT50Q-1M
- added D1, D2: 19-213/Y2C-CQ2R2L/3T(CY), LEDs:LED_0603_HandSoldering, symbol Device:LED
- added J2, J3: Conn_01x08_Female, Connectors_JST:JST_PH_B8B-PH-SM4-TB_08x2.00mm_Straight, symbol Connector:Conn_01x08_Female
- added R1, R2: 100, Resistor_SMD:R_0603_1608Metric_Pad0.84x1.00mm_HandSolder, symbol Device:R
- added TP1: VBATT_OUT, TestPoint:TestPoint_Loop_D1.80mm_Drill1.0mm_Beaded, symbol Connector:TestPoint
- added TP10: SWDIO, TestPoint:TestPoint_Loop_D1.80mm_Drill1.0mm_Beaded, symbol Connector:TestPoint
- added TP11: NFC1, TestPoint:TestPoint_Loop_D1.80mm_Drill1.0mm_Beaded, symbol Connector:TestPoint
- added TP12: SWDCLK, TestPoint:TestPoint_Loop_D1.80mm_Drill1.0mm_Beaded, symbol Connector:TestPoint
- added TP13: NFC2, TestPoint:TestPoint_Loop_D1.80mm_Drill1.0mm_Beaded, symbol Connector:TestPoint
- added TP14: MISO, TestPoint:TestPoint_Loop_D1.80mm_Drill1.0mm_Beaded, symbol Connector:TestPoint
- added TP15: MOSI, TestPoint:TestPoint_Loop_D1.80mm_Drill1.0mm_Beaded, symbol Connector:TestPoint
- added TP16: SCK, TestPoint:TestPoint_Loop_D1.80mm_Drill1.0mm_Beaded, symbol Connector:TestPoint
- added TP17: ~CS0, TestPoint:TestPoint_Loop_D1.80mm_Drill1.0mm_Beaded, symbol Connector:TestPoint
- added TP18: ~CS1, TestPoint:TestPoint_Loop_D1.80mm_Drill1.0mm_Beaded, symbol Connector:TestPoint
- added TP19: ~EOC0, TestPoint:TestPoint_Loop_D1.80mm_Drill1.0mm_Beaded, symbol Connector:TestPoint
- added TP2: AIN5, TestPoint:TestPoint_Loop_D1.80mm_Drill1.0mm_Beaded, symbol Connector:TestPoint
- added TP20: EOC1, TestPoint:TestPoint_Loop_D1.80mm_Drill1.0mm_Beaded, symbol Connector:TestPoint
- added TP21: AREF, TestPoint:TestPoint_Loop_D1.80mm_Drill1.0mm_Beaded, symbol Connector:TestPoint
- added TP22: H0, TestPoint:TestPoint_Loop_D1.80mm_Drill1.0mm_Beaded, symbol Connector:TestPoint
- added TP23: H1, TestPoint:TestPoint_Loop_D1.80mm_Drill1.0mm_Beaded, symbol Connector:TestPoint
- added TP3: AIN0, TestPoint:TestPoint_Loop_D1.80mm_Drill1.0mm_Beaded, symbol Connector:TestPoint
- added TP4: AIN7, TestPoint:TestPoint_Loop_D1.80mm_Drill1.0mm_Beaded, symbol Connector:TestPoint
- added TP5: AIN4, TestPoint:TestPoint_Loop_D1.80mm_Drill1.0mm_Beaded, symbol Connector:TestPoint
- added TP6: AIN6, TestPoint:TestPoint_Loop_D1.80mm_Drill1.0mm_Beaded, symbol Connector:TestPoint
- added TP7: AIN2, TestPoint:TestPoint_Loop_D1.80mm_Drill1.0mm_Beaded, symbol Connector:TestPoint
- added TP8: AIN3, TestPoint:TestPoint_Loop_D1.80mm_Drill1.0mm_Beaded, symbol Connector:TestPoint
- added TP9: SWDI, TestPoint:TestPoint_Loop_D1.80mm_Drill1.0mm_Beaded, symbol Connector:TestPoint
- added U3: 113990582, SamacSys_Parts:113990582, symbol SamacSys_Parts:113990582
- C1: renamed from C2; footprint Capacitor_SMD:C_0603_1608Metric_Pad1.08x0.95mm_HandSolder -> Capacitors_SMD:C_0603_HandSoldering
- C2: renamed from C4; footprint Inductor_SMD:L_0402_1005Metric_Pad0.77x0.64mm_HandSolder -> Capacitor_SMD:C_0402_1005Metric
- C3: renamed from C5; footprint Inductor_SMD:L_0402_1005Metric_Pad0.77x0.64mm_HandSolder -> Capacitor_SMD:C_0402_1005Metric
- C4: renamed from C1; footprint Capacitor_SMD:C_0603_1608Metric_Pad1.08x0.95mm_HandSolder -> Capacitors_SMD:C_0603_HandSoldering
- J1: footprint (none) -> WARG:USB_Micro-B_10118194-0001LF
- L1: footprint Inductor_SMD:L_0805_2012Metric_Pad1.15x1.40mm_HandSolder -> Inductors_SMD:L_0805_HandSoldering
- R3: renamed from R1; footprint Resistor_SMD:R_0603_1608Metric -> Resistor_SMD:R_0603_1608Metric_Pad0.84x1.00mm_HandSolder
- R4: renamed from R2; footprint Resistor_SMD:R_0603_1608Metric -> Resistor_SMD:R_0603_1608Metric_Pad0.84x1.00mm_HandSolder
- R5: renamed from R3; footprint (none) -> Resistor_SMD:R_0603_1608Metric_Pad0.84x1.00mm_HandSolder
- S1: footprint digikey-footprints:PushButton_12x12mm_THT_GPTS203211B -> SamacSys_Parts:GPTS203211B; symbol dk_Pushbutton-Switches:GPTS203211B -> Glove-PCB-rescue:GPTS203211B-dk_Pushbutton-Switches
- XTAL1: footprint digikey-footprints:SMD-2_3.2x1.5mm -> SamacSys_Parts:ECX-31B; symbol dk_Crystals:ECS-_327-12_5-34B-TR -> Glove-PCB-rescue:ECS-_327-12_5-34B-TR-dk_Crystals
Connections:
- net labels added: +3.3V, AREF, H0, H1, LED0, LED1, VBATT_OUT, VBUS, VDD, ~CS0, ~EOC0, ~EOC1
- net labels removed: 5V, VBatt, VCC1, ~CS2
- wire segments 59 -> 126
- no-connect marks 0 -> 28
Other:
- moved on the sheet: C1, C2, C3, C4, J1, L1, R3, R4, R5

Commit message: Added project and digikey footprints. Added mini-spox connectors.
Parts:
- removed J2, J3: Conn_01x08_Female, Connectors_JST:JST_PH_B8B-PH-SM4-TB_08x2.00mm_Straight, symbol Connector:Conn_01x08_Female
- added J2, J5: Conn_01x06_Female, Glove-PCB:22-05-7065, symbol Connector:Conn_01x06_Female
- added J3: Conn_01x04_Female, Glove-PCB:22-05-7045, symbol Connector:Conn_01x04_Female
- TP1, TP10, TP11, TP12, TP13, TP14, TP15, TP16, TP17, TP18, TP19, TP2, TP20, TP21, TP22, TP23, TP3, TP4, TP5, TP6, TP7, TP8, TP9: footprint TestPoint:TestPoint_Loop_D1.80mm_Drill1.0mm_Beaded -> TestPoint:TestPoint_Pad_D1.5mm
Changed lines of the file:
@@
 F 1 "USB_B_Micro" H 7500 1400 50  0000 L CNN
 F 2 "WARG:USB_Micro-B_10118194-0001LF" H 7550 1800 50  0001 C CNN
-F 3 "~" H 7550 1800 50  0001 C CNN
+F 3 "https://www.amphenol-icc.com/media/wysiwyg/files/drawing/10118194.pdf" H 7550 1800 50  0001 C CNN
 	1    7400 1850
 	-1   0    0    1
@@
 Text Label 7450 5350 2    50   ~ 0
 H0
-$Comp
-L Connector:Conn_01x08_Female J2
-U 1 1 5FF78DC1
-P 9950 4400
-F 0 "J2" H 9978 4376 50  0000 L CNN
-F 1 "Conn_01x08_Female" H 9978 4285 50  0000 L CNN
-F 2 "Connectors_JST:JST_PH_B8B-PH-SM4-TB_08x2.00mm_Straight" H 9950 4400 50  0001 C CNN
-F 3 "~" H 9950 4400 50  0001 C CNN
-	1    9950 4400
-	1    0    0    -1
-$EndComp
 Wire Wire Line
 	4300 1750 3950 1750
@@
 LED1
 $Comp
-L Connector:Conn_01x08_Female J3
-U 1 1 5FFD7598
-P 9950 5200
-F 0 "J3" H 9978 5176 50  0000 L CNN
-F 1 "Conn_01x08_Female" H 9978 5085 50  0000 L CNN
-F 2 "Connectors_JST:JST_PH_B8B-PH-SM4-TB_08x2.00mm_Straight" H 9950 5200 50  0001 C CNN
-F 3 "~" H 9950 5200 50  0001 C CNN
-	1    9950 5200
-	1    0    0    -1
-$EndComp
-$Comp
 L Connector:TestPoint TP14
 U 1 1 5FFF8A11
@@
 F 0 "TP14" V 7300 4600 50  0000 C CNN
 F 1 "MISO" V 7300 4400 50  0000 C CNN
-F 2 "TestPoint:TestPoint_Loop_D1.80mm_Drill1.0mm_Beaded" H 7500 4100 50  0001 C CNN
+F 2 "TestPoint:TestPoint_Pad_D1.5mm" H 7500 4100 50  0001 C CNN
 F 3 "~" H 7500 4100 50  0001 C CNN
 	1    7300 4100
@@
 F 0 "TP15" V 7300 4700 50  0000 C CNN
 F 1 "MOSI" V 7300 4500 50  0000 C CNN
-F 2 "TestPoint:TestPoint_Loop_D1.80mm_Drill1.0mm_Beaded" H 7500 4200 50  0001 C CNN
+F 2 "TestPoint:TestPoint_Pad_D1.5mm" H 7500 4200 50  0001 C CNN
 F 3 "~" H 7500 4200 50  0001 C CNN
 	1    7300 4200
@@
 F 0 "TP16" V 7300 4800 50  0000 C CNN
 F 1 "SCK" V 7300 4600 50  0000 C CNN
-F 2 "TestPoint:TestPoint_Loop_D1.80mm_Drill1.0mm_Beaded" H 7500 4300 50  0001 C CNN
+F 2 "TestPoint:TestPoint_Pad_D1.5mm" H 7500 4300 50  0001 C CNN
 F 3 "~" H 7500 4300 50  0001 C CNN
 	1    7300 4300
@@
 F 0 "TP17" V 7300 4900 50  0000 C CNN
 F 1 "~CS0" V 7300 4700 50  0000 C CNN
-F 2 "TestPoint:TestPoint_Loop_D1.80mm_Drill1.0mm_Beaded" H 7500 4400 50  0001 C CNN
+F 2 "TestPoint:TestPoint_Pad_D1.5mm" H 7500 4400 50  0001 C CNN
 F 3 "~" H 7500 4400 50  0001 C CNN
 	1    7300 4400
@@
 F 0 "TP18" V 7300 5000 50  0000 C CNN
 F 1 "~CS1" V 7300 4800 50  0000 C CNN
-F 2 "TestPoint:TestPoint_Loop_D1.80mm_Drill1.0mm_Beaded" H 7500 4500 50  0001 C CNN
+F 2 "TestPoint:TestPoint_Pad_D1.5mm" H 7500 4500 50  0001 C CNN
 F 3 "~" H 7500 4500 50  0001 C CNN
 	1    7300 4500
@@
 F 0 "TP19" V 7300 5200 50  0000 C CNN
 F 1 "~EOC0" V 7300 5000 50  0000 C CNN
-F 2 "TestPoint:TestPoint_Loop_D1.80mm_Drill1.0mm_Beaded" H 7500 4700 50  0001 C CNN
+F 2 "TestPoint:TestPoint_Pad_D1.5mm" H 7500 4700 50  0001 C CNN
 F 3 "~" H 7500 4700 50  0001 C CNN
 	1    7300 4700
@@
 F 0 "TP20" V 7300 5300 50  0000 C CNN
 F 1 "EOC1" V 7300 5100 50  0000 C CNN
-F 2 "TestPoint:TestPoint_Loop_D1.80mm_Drill1.0mm_Beaded" H 7500 4800 50  0001 C CNN
+F 2 "TestPoint:TestPoint_Pad_D1.5mm" H 7500 4800 50  0001 C CNN
 F 3 "~" H 7500 4800 50  0001 C CNN
 	1    7300 4800
@@
 F 0 "TP22" V 7300 5850 50  0000 C CNN
 F 1 "H0" V 7300 5650 50  0000 C CNN
-F 2 "TestPoint:TestPoint_Loop_D1.80mm_Drill1.0mm_Beaded" H 7500 5350 50  0001 C CNN
+F 2 "TestPoint:TestPoint_Pad_D1.5mm" H 7500 5350 50  0001 C CNN
 F 3 "~" H 7500 5350 50  0001 C CNN
 	1    7300 5350
@@
 F 0 "TP23" V 7300 6200 50  0000 C CNN
 F 1 "H1" V 7300 6000 50  0000 C CNN
-F 2 "TestPoint:TestPoint_Loop_D1.80mm_Drill1.0mm_Beaded" H 7500 5700 50  0001 C CNN
+F 2 "TestPoint:TestPoint_Pad_D1.5mm" H 7500 5700 50  0001 C CNN
 F 3 "~" H 7500 5700 50  0001 C CNN
 	1    7300 5700
@@
 F 0 "TP9" V 6350 3550 50  0000 C CNN
 F 1 "SWDI" V 6350 3350 50  0000 C CNN
-F 2 "TestPoint:TestPoint_Loop_D1.80mm_Drill1.0mm_Beaded" H 6550 3050 50  0001 C CNN
+F 2 "TestPoint:TestPoint_Pad_D1.5mm" H 6550 3050 50  0001 C CNN
 F 3 "~" H 6550 3050 50  0001 C CNN
 	1    6350 3050
@@
 F 0 "TP12" V 6350 4250 50  0000 C CNN
 F 1 "SWDCLK" V 6350 4000 50  0000 C CNN
-F 2 "TestPoint:TestPoint_Loop_D1.80mm_Drill1.0mm_Beaded" H 6550 3650 50  0001 C CNN
+F 2 "TestPoint:TestPoint_Pad_D1.5mm" H 6550 3650 50  0001 C CNN
 F 3 "~" H 6550 3650 50  0001 C CNN
 	1    6350 3650
@@
 F 0 "TP10" V 6350 3950 50  0000 C CNN
 F 1 "SWDIO" V 6350 3750 50  0000 C CNN
-F 2 "TestPoint:TestPoint_Loop_D1.80mm_Drill1.0mm_Beaded" H 6550 3450 50  0001 C CNN
+F 2 "TestPoint:TestPoint_Pad_D1.5mm" H 6550 3450 50  0001 C CNN
 F 3 "~" H 6550 3450 50  0001 C CNN
 	1    6350 3450
@@
 F 0 "TP21" V 7300 5600 50  0000 C CNN
 F 1 "AREF" V 7300 5400 50  0000 C CNN
-F 2 "TestPoint:TestPoint_Loop_D1.80mm_Drill1.0mm_Beaded" H 7500 5100 50  0001 C CNN
+F 2 "TestPoint:TestPoint_Pad_D1.5mm" H 7500 5100 50  0001 C CNN
 F 3 "~" H 7500 5100 50  0001 C CNN
 	1    7300 5100
@@
 	1    0    0    -1
 $EndComp
-Text Label 3950 2550 0    50   ~ 0
-AREF
 Wire Wire Line
 	6350 2450 6000 2450
@@
 F 0 "TP13" V 6350 4350 50  0000 C CNN
 F 1 "NFC2" V 6350 4100 50  0000 C CNN
-F 2 "TestPoint:TestPoint_Loop_D1.80mm_Drill1.0mm_Beaded" H 6550 3750 50  0001 C CNN
+F 2 "TestPoint:TestPoint_Pad_D1.5mm" H 6550 3750 50  0001 C CNN
 F 3 "~" H 6550 3750 50  0001 C CNN
 	1    6350 3750
@@
 F 0 "TP11" V 6350 4150 50  0000 C CNN
 F 1 "NFC1" V 6350 3900 50  0000 C CNN
-F 2 "TestPoint:TestPoint_Loop_D1.80mm_Drill1.0mm_Beaded" H 6550 3550 50  0001 C CNN
+F 2 "TestPoint:TestPoint_Pad_D1.5mm" H 6550 3550 50  0001 C CNN
 F 3 "~" H 6550 3550 50  0001 C CNN
 	1    6350 3550
@@
 F 0 "TP1" V 2800 7350 50  0000 C CNN
 F 1 "VBATT_OUT" V 2800 7000 50  0000 C CNN
-F 2 "TestPoint:TestPoint_Loop_D1.80mm_Drill1.0mm_Beaded" H 3000 6600 50  0001 C CNN
+F 2 "TestPoint:TestPoint_Pad_D1.5mm" H 3000 6600 50  0001 C CNN
 F 3 "~" H 3000 6600 50  0001 C CNN
 	1    2800 6600
@@
 F 0 "TP7" V 3950 3950 50  0000 C CNN
 F 1 "AIN2" V 3950 3750 50  0000 C CNN
-F 2 "TestPoint:TestPoint_Loop_D1.80mm_Drill1.0mm_Beaded" H 4150 3450 50  0001 C CNN
+F 2 "TestPoint:TestPoint_Pad_D1.5mm" H 4150 3450 50  0001 C CNN
 F 3 "~" H 4150 3450 50  0001 C CNN
 	1    3950 3450
@@
 F 0 "TP8" V 3950 4050 50  0000 C CNN
 F 1 "AIN3" V 3950 3850 50  0000 C CNN
-F 2 "TestPoint:TestPoint_Loop_D1.80mm_Drill1.0mm_Beaded" H 4150 3550 50  0001 C CNN
+F 2 "TestPoint:TestPoint_Pad_D1.5mm" H 4150 3550 50  0001 C CNN
 F 3 "~" H 4150 3550 50  0001 C CNN
 	1    3950 3550
@@
 F 0 "TP2" V 3950 2950 50  0000 C CNN
 F 1 "AIN5" V 3950 2750 50  0000 C CNN
-F 2 "TestPoint:TestPoint_Loop_D1.80mm_Drill1.0mm_Beaded" H 4150 2450 50  0001 C CNN
+F 2 "TestPoint:TestPoint_Pad_D1.5mm" H 4150 2450 50  0001 C CNN
 F 3 "~" H 4150 2450 50  0001 C CNN
 	1    3950 2450
@@
 F 0 "TP3" V 3950 3050 50  0000 C CNN
 F 1 "AIN0" V 3950 2850 50  0000 C CNN
-F 2 "TestPoint:TestPoint_Loop_D1.80mm_Drill1.0mm_Beaded" H 4150 2550 50  0001 C CNN
+F 2 "TestPoint:TestPoint_Pad_D1.5mm" H 4150 2550 50  0001 C CNN
 F 3 "~" H 4150 2550 50  0001 C CNN
 	1    3950 2550
@@
 F 0 "TP4" V 3950 3150 50  0000 C CNN
 F 1 "AIN7" V 3950 2950 50  0000 C CNN
-F 2 "TestPoint:TestPoint_Loop_D1.80mm_Drill1.0mm_Beaded" H 4150 2650 50  0001 C CNN
+F 2 "TestPoint:TestPoint_Pad_D1.5mm" H 4150 2650 50  0001 C CNN
 F 3 "~" H 4150 2650 50  0001 C CNN
 	1    3950 2650
@@
 F 0 "TP5" V 3950 3250 50  0000 C CNN
 F 1 "AIN4" V 3950 3050 50  0000 C CNN
-F 2 "TestPoint:TestPoint_Loop_D1.80mm_Drill1.0mm_Beaded" H 4150 2750 50  0001 C CNN
+F 2 "TestPoint:TestPoint_Pad_D1.5mm" H 4150 2750 50  0001 C CNN
 F 3 "~" H 4150 2750 50  0001 C CNN
 	1    3950 2750
@@
 F 0 "TP6" V 3950 3350 50  0000 C CNN
 F 1 "AIN6" V 3950 3150 50  0000 C CNN
-F 2 "TestPoint:TestPoint_Loop_D1.80mm_Drill1.0mm_Beaded" H 4150 2850 50  0001 C CNN
+F 2 "TestPoint:TestPoint_Pad_D1.5mm" H 4150 2850 50  0001 C CNN
 F 3 "~" H 4150 2850 50  0001 C CNN
 	1    3950 2850
@@
 NoConn ~ 3950 1850
 NoConn ~ 7100 1650
+$Comp
+L Connector:Conn_01x04_Female J3
+U 1 1 5FC920AE
+P 9950 4800
+F 0 "J3" H 9978 4776 50  0000 L CNN
+F 1 "Conn_01x04_Female" H 9978 4685 50  0000 L CNN
+F 2 "Glove-PCB:22-05-7045" H 9950 4800 50  0001 C CNN
+F 3 "~" H 9950 4800 50  0001 C CNN
+	1    9950 4800
+	1    0    0    -1
+$EndComp
+$Comp
+L Connector:Conn_01x06_Female J2
+U 1 1 5FC937C0
+P 9950 4300
+F 0 "J2" H 9978 4276 50  0000 L CNN
+F 1 "Conn_01x06_Female" H 9978 4185 50  0000 L CNN
+F 2 "Glove-PCB:22-05-7065" H 9950 4300 50  0001 C CNN
+F 3 "~" H 9950 4300 50  0001 C CNN
+	1    9950 4300
+	1    0    0    -1
+$EndComp
+$Comp
+L Connector:Conn_01x06_Female J5
+U 1 1 5FC94656
+P 9950 5300
+F 0 "J5" H 9978 5276 50  0000 L CNN
+F 1 "Conn_01x06_Female" H 9978 5185 50  0000 L CNN
+F 2 "Glove-PCB:22-05-7065" H 9950 5300 50  0001 C CNN
+F 3 "~" H 9950 5300 50  0001 C CNN
+	1    9950 5300
+	1    0    0    -1
+$EndComp
 $EndSCHEMATC

Commit message: Placement done. Started layout.
Parts:
- removed S1: GPTS203211B, SamacSys_Parts:GPTS203211B, symbol Glove-PCB-rescue:GPTS203211B-dk_Pushbutton-Switches
- removed TP2: AIN5, TestPoint:TestPoint_Pad_D1.5mm, symbol Connector:TestPoint
- removed TP3: AIN0, TestPoint:TestPoint_Pad_D1.5mm, symbol Connector:TestPoint
- removed TP4: AIN7, TestPoint:TestPoint_Pad_D1.5mm, symbol Connector:TestPoint
- removed TP5: AIN4, TestPoint:TestPoint_Pad_D1.5mm, symbol Connector:TestPoint
- removed TP6: AIN6, TestPoint:TestPoint_Pad_D1.5mm, symbol Connector:TestPoint
- removed TP7: AIN2, TestPoint:TestPoint_Pad_D1.5mm, symbol Connector:TestPoint
- removed TP8: AIN3, TestPoint:TestPoint_Pad_D1.5mm, symbol Connector:TestPoint
- added SW1: TS-1109S-B-B, Glove-PCB:Button, symbol Glove_PCB:SW_Push_Dual_1-2short_3-4short
- renumbered TP22 to TP1, TP16 to TP10, TP17 to TP11, TP18 to TP12, TP19 to TP13, TP20 to TP14, TP21 to TP15, TP1 to TP16, TP23 to TP2, TP9 to TP3, TP10 to TP4, TP11 to TP5, TP12 to TP6, TP13 to TP7, TP14 to TP8, TP15 to TP9
Connections:
- net labels added: NFC1, NFC2, SWDCLK, SWDI, SWDIO
- wire segments 126 -> 132
- no-connect marks 28 -> 35
